Commit message: Add RL deployment nodes

File: src/doggy/robot.urdf (robot description, URDF)
Before this commit: robot doggy, 5 links, 4 joints
Links:
- added link FL_foot, mass 1e-9
- added link FR_foot, mass 1e-9
- added link RL_foot, mass 1e-9
- added link RR_foot, mass 1e-9
- added link base_link, mass 1e-9
- added link calf_2, mass 0.023; collision mesh filename=package://assets/foot.stl; collision mesh filename=package://assets/foot_tip.stl
- added link calf_3, mass 0.023; collision mesh filename=package://assets/foot.stl; collision mesh filename=package://assets/foot_tip.stl
- added link calf_4, mass 0.023; collision mesh filename=package://assets/foot.stl; collision mesh filename=package://assets/foot_tip.stl
- added link hipjoint_2, mass 0.0326833; collision mesh filename=package://assets/feetech_sts2032_20g__2.stl; collision mesh filename=package://assets/hipjoint_v4.stl
- added link hipjoint_mir, mass 0.0326833; collision mesh filename=package://assets/feetech_sts2032_20g__2.stl; collision mesh filename=package://assets/hipjoint_v4__2.stl
- added link hipjoint_mir_2, mass 0.0326833; collision mesh filename=package://assets/feetech_sts2032_20g__2.stl; collision mesh filename=package://assets/hipjoint_v4__2.stl
- added link imu, mass 1e-9
- added link linkage_a_v2_0713_mir_2, mass 0.00221365; collision mesh filename=package://assets/linkage_a_v2_0713_mir.stl; visual mesh filename=package://assets/linkage_a_v2_0713_mir.stl
- added link linkage_a_v2_0713_mir_3, mass 0.00221365; collision mesh filename=package://assets/linkage_a_v2_0713_mir.stl; visual mesh filename=package://assets/linkage_a_v2_0713_mir.stl
- added link linkage_a_v2_0713_mir_4, mass 0.00221365; collision mesh filename=package://assets/linkage_a_v2_0713_mir.stl; visual mesh filename=package://assets/linkage_a_v2_0713_mir.stl
- added link thigh, mass 0.0619252; collision mesh filename=package://assets/feetech_sts2032_20g__3.stl; collision mesh filename=package://assets/inner_leg_v4.stl
- added link thigh_2, mass 0.0619252; collision mesh filename=package://assets/feetech_sts2032_20g__3.stl; collision mesh filename=package://assets/inner_leg_v4.stl
- added link thigh_mir_2, mass 0.0369251; collision mesh filename=package://assets/feetech_sts2032_20g_mir1.stl; collision mesh filename=package://assets/inner_leg_v4_mirrored.stl
Joints:
- added joint FL_foot_frame: type fixed, parent calf_2, child FL_foot, origin xyz=-3e-06 0.0919 -0.006 rpy=-1.5708 -5.14606e-32 3.14159, axis 0 0 0
- added joint FL_hip_pitch: type revolute, parent hipjoint_mir, child thigh_mir_2, origin xyz=1.25767e-17 -0.0187 -0.0117 rpy=1.5708 -9.36772e-31 -3.14159, axis 0 0 1, limit lower=-1.5708 upper=0.174533 effort=10 velocity=10
- added joint FL_hip_roll: type revolute, parent body, child hipjoint_mir, origin xyz=-0.125 -0.036 -0.00279 rpy=-1.51223e-15 1.5708 0, axis 0 0 1, limit lower=-0.174533 upper=0.349066 effort=10 velocity=10
- added joint FL_knee: type revolute, parent thigh_mir_2, child calf_2, origin xyz=2.30081e-13 -0.08 -0.006 rpy=-6.70532e-30 -7.2455e-30 1.5708, axis 0 0 1, limit lower=-1.309 upper=1.5708 effort=10 velocity=10
- added joint FL_motor3: type revolute, parent thigh_mir_2, child linkage_a_v2_0713_mir_2, origin xyz=0.0147 0 -0.011 rpy=-1.5708 6.89354e-17 1.5708, axis 0 0 1, limit lower=-1.0472 upper=1.48353 effort=10 velocity=10
- added joint FR_foot_frame: type fixed, parent calf_3, child FR_foot, origin xyz=-3e-06 -0.0919 -0.006 rpy=1.5708 5.52464e-33 3.14159, axis 0 0 0
- added joint FR_hip_pitch: type revolute, parent hipjoint_2, child thigh, origin xyz=-1.01048e-16 0.0187 -0.0117 rpy=-1.5708 8.48025e-30 -3.14159, axis 0 0 1, limit lower=-0.174533 upper=1.5708 effort=10 velocity=10
- added joint FR_hip_roll: type revolute, parent body, child hipjoint_2, origin xyz=-0.125 0.036 -0.00279 rpy=-6.89354e-17 1.5708 0, axis 0 0 1, limit lower=-0.349066 upper=0.174533 effort=10 velocity=10
- added joint FR_knee: type revolute, parent thigh, child calf_3, origin xyz=2.29983e-13 0.08 -0.006 rpy=3.36134e-27 -4.48177e-28 -1.5708, axis 0 0 1, limit lower=-1.309 upper=1.5708 effort=10 velocity=10
- added joint FR_motor3: type revolute, parent thigh, child linkage_a_v2_0713_mir_3, origin xyz=0.0147 0 -0.011 rpy=-1.5708 6.16791e-17 1.5708, axis 0 0 1, limit lower=-1.48353 upper=1.0472 effort=10 velocity=10
- added joint RL_foot_frame: type fixed, parent calf, child RL_foot, origin xyz=-3e-06 0.0919 -0.005 rpy=-1.5708 1.27732e-31 3.14159, axis 0 0 0
- added joint RR_foot_frame: type fixed, parent calf_4, child RR_foot, origin xyz=-3e-06 -0.0919 -0.006 rpy=1.5708 -1.39172e-31 3.14159, axis 0 0 0
- added joint RR_hip_pitch: type revolute, parent hipjoint_mir_2, child thigh_2, origin xyz=1.25767e-17 -0.0187 -0.0117 rpy=1.5708 -3.24173e-30 3.14159, axis 0 0 1, limit lower=-0.174533 upper=1.5708 effort=10 velocity=10
- added joint RR_hip_roll: type revolute, parent body, child hipjoint_mir_2, origin xyz=0.125 0.036 -0.00279 rpy=3.14159 1.5708 0, axis 0 0 1, limit lower=-0.174533 upper=0.349066 effort=10 velocity=10
- added joint RR_knee: type revolute, parent thigh_2, child calf_4, origin xyz=2.30041e-13 0.08 -0.006 rpy=-1.49884e-29 4.87234e-30 -1.5708, axis 0 0 1, limit lower=-1.5708 upper=1.309 effort=10 velocity=10
- added joint RR_motor3: type revolute, parent thigh_2, child linkage_a_v2_0713_mir_4, origin xyz=0.0181 -5.55112e-17 -0.011 rpy=-1.5708 6.16791e-17 1.5708, axis 0 0 1, limit lower=-1.48353 upper=1.0472 effort=10 velocity=10
- added joint base_link_frame: type fixed, parent body, child base_link, origin xyz=-2.89644e-18 -2.35336e-18 0.003 rpy=-3.24138e-43 -8.96831e-44 -3.14159, axis 0 0 0
- added joint imu_frame: type fixed, parent body, child imu, origin xyz=-2.89644e-18 -2.1684e-18 -0.0145 rpy=0 -0 3.14159, axis 0 0 0
- joint RL_hip_pitch: origin xyz=-1.17961e-16 0.0187 -0.0117 rpy=-1.5708 -2.22459e-28 -3.14159 -> xyz=-1.11022e-16 0.0187 -0.0117 rpy=-1.5708 -3.06162e-16 -3.14159
- joint RL_hip_roll: limit lower=-0.174533 upper=0.349066 effort=10 velocity=10 -> lower=-0.349066 upper=0.174533 effort=10 velocity=10; origin xyz=0.125 -0.036 0.02471 rpy=-3.14159 1.5708 0 -> xyz=0.125 -0.036 -0.00279 rpy=-3.14159 1.5708 0
- joint RL_knee: origin xyz=2.30083e-13 -0.08 -0.007 rpy=-6.53674e-26 -8.38583e-27 1.5708 -> xyz=2.30043e-13 -0.08 -0.007 rpy=6.12323e-17 -6.30424e-31 1.5708
- joint RL_motor3: origin xyz=0.0181 5.55112e-17 -0.011 rpy=-1.5708 9.6691e-17 1.5708 -> xyz=0.0181 2.77556e-17 -0.011 rpy=-1.5708 2.19156e-16 1.5708

Commit message: urdf editted

File: src/doggy/robot.urdf (robot description, URDF)
Before this commit: robot doggy, 23 links, 22 joints
Links:
- removed link linkage_a_v2_0713_mir
- removed link linkage_a_v2_0713_mir_2
- removed link linkage_a_v2_0713_mir_3
- removed link linkage_a_v2_0713_mir_4
Joints:
- removed joint FL_motor3
- removed joint FR_motor3
- removed joint RL_motor3
- removed joint RR_motor3
